File: EAGLE/vr42/vr42-revA.brd (EAGLE design)
At the start: 227.6 x 74.2 mm, 197 parts, among them Q1 2N7002, Q2 DMG2305UX-7, U1 STM32F405RGT6, U10 74HC589A_DT, U2 USB3300-EZK, U3 TS3USB221A-Q1, U4 TPS2553DBVR-1, U4X M25C, U5 74HC589A_DT, U6 74HC589A_DT, U7 74HC589A_DT, U8 74HC589A_DT, U9 74HC589A_DT, Y1 32.768kHz ±20ppm 6pF, Y2 25MHz 9pF, Y3 24MHz

Commit message: .
Parts:
- removed U$14: 74AHCT1G125GW, ts_keyboards:SC-88A__TSSOP5__SOT353-1
- removed U10, U5, U6, U7, U8, U9: 74HC589A_DT, __untitled:TSSOP16
- added I1: SK6812-E-REVERSE, ts_keyboards:SK6812-E-MILL
- added I44: ARGB, __temp_to_delete:ARGB
- added LS: 74AHCT1G125GW, ts_keyboards:SC-88A__TSSOP5__SOT353-1
- added M0, M1, M2, M3, M4, M5: 74HC589A_DT, __untitled:TSSOP16
- added U$2, U$3: MOLEX_0781710005, molex-pico-ezmate:MOLEX_781710005
- added U$4, U$5: MOLEX_0781710003, molex-pico-ezmate:MOLEX_781710003
- added U$6: VR42_MLB_FOOTPRINT, __temp_to_delete:VR42_MLB_FOOTPRINT
- added U$7: UBD_FOOTPRINT, __temp_to_delete:UDB_FOOTPRINT
- C16, C17: value 2.2pF -> 0.1uF
- C20: value 100nF -> 22uF
- C22: value 22uF -> 100nF
- C25, C26: value 0.1uF -> 2.2pF
- U$1: value ARGB -> VR42_MLB_FOOTPRINT; device __temp_to_delete:ARGB -> __temp_to_delete:VR42_MLB_FOOTPRINT
- moved C30 220.5 mm to (252.0, 5.00), turned to 270 degrees
- moved C19 212.4 mm to (258.0, 35.0)
- moved C18 203.1 mm to (258.0, 45.0)
- moved R28 202.4 mm to (245.5, 62.0), turned to 90 degrees
- moved UDB2 202.3 mm to (246.0, 7.60)
- moved C47 200.3 mm to (5.00, 29.0)
- moved C31 199.3 mm to (253.0, 73.0), turned to 270 degrees
- moved R26 199.1 mm to (234.0, 24.0)
- moved C48 194.5 mm to (5.00, 26.0)
- moved C49 189.0 mm to (5.00, 23.0)
- moved C22 186.8 mm to (243.0, 17.0), turned to 90 degrees
- moved C23 184.3 mm to (238.0, 20.0), turned to 180 degrees
- moved C24 184.1 mm to (234.0, 20.0)
- moved C50 183.6 mm to (5.00, 20.0)
- moved C20 180.0 mm to (238.0, 10.0), turned to 180 degrees
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- renumbered Z1 to I32, Z10 to I41, Z11 to I42, Z12 to I43, Z13 to I21, Z14 to I22, Z15 to I23, Z16 to I24, Z17 to I25, Z18 to I26, Z19 to I27, Z2 to I33, Z20 to I28, Z21 to I29, Z22 to I30, Z23 to I31, Z24 to I10, Z25 to I11, Z26 to I12, Z27 to I13, Z28 to I14, Z29 to I15, Z3 to I34, Z30 to I16, Z31 to I17, Z32 to I18, Z33 to I19, Z34 to I20, Z35 to I2, Z36 to I3, Z37 to I4, Z38 to I5, Z39 to I6, Z4 to I35, Z40 to I7, Z41 to I8, Z42 to I9, Z5 to I36, Z6 to I37, Z7 to I38, Z8 to I39, Z9 to I40
Connections:
- removed net N$1: C1.1, U1.47
- removed net N$2: C2.1, U1.31
- removed net N$39: I21.4-DIN, I43.2-DOUT
- removed net N$61: I2.4-DIN, I20.2-DOUT
- removed net SK6803: I32.4-DIN, R12.1
- removed net SK6803_PWR: C46.1, C47.1, C48.1, C49.1, C50.1, I10.1-VDD, I11.1-VDD, I12.1-VDD, I13.1-VDD, I14.1-VDD, I15.1-VDD, I16.1-VDD, I17.1-VDD, I18.1-VDD, I19.1-VDD, I2.1-VDD, I20.1-VDD, I21.1-VDD, I22.1-VDD, I23.1-VDD, I24.1-VDD, I25.1-VDD, I26.1-VDD, I27.1-VDD, I28.1-VDD, I29.1-VDD, I3.1-VDD, I30.1-VDD, I31.1-VDD, I32.1-VDD, I33.1-VDD, I34.1-VDD, I35.1-VDD, I36.1-VDD, I37.1-VDD, I38.1-VDD, I39.1-VDD, I4.1-VDD, I40.1-VDD, I41.1-VDD, I42.1-VDD, I43.1-VDD, I5.1-VDD, I6.1-VDD, I7.1-VDD, I8.1-VDD, I9.1-VDD, U$1.V, U$14.6, U4.6
- new net ARGB_5V_D: I1.4-DIN, R12.1
- new net ARGB_PWR: C44.1, C46.1, C47.1, C48.1, C49.1, C50.1, I1.1-VDD, I10.1-VDD, I11.1-VDD, I12.1-VDD, I13.1-VDD, I14.1-VDD, I15.1-VDD, I16.1-VDD, I17.1-VDD, I18.1-VDD, I19.1-VDD, I2.1-VDD, I20.1-VDD, I21.1-VDD, I22.1-VDD, I23.1-VDD, I24.1-VDD, I25.1-VDD, I26.1-VDD, I27.1-VDD, I28.1-VDD, I29.1-VDD, I3.1-VDD, I30.1-VDD, I31.1-VDD, I32.1-VDD, I33.1-VDD, I34.1-VDD, I35.1-VDD, I36.1-VDD, I37.1-VDD, I38.1-VDD, I39.1-VDD, I4.1-VDD, I40.1-VDD, I41.1-VDD, I42.1-VDD, I43.1-VDD, I44.V, I5.1-VDD, I6.1-VDD, I7.1-VDD, I8.1-VDD, I9.1-VDD, LS.6, U$4.2, U$5.2, U4.6
- new net N$36: I31.2-DOUT, I32.4-DIN
- new net N$37: I43.2-DOUT, I44.D
- new net N$46: I1.2-DOUT, I2.4-DIN
- new net VCAP_1: C1.1, U1.31
- new net VCAP_2: C2.1, U1.47
- net ARGB_D: now also U$4.3, U$5.3
- net GND: now also C16.2, C17.2, C25.1, C26.1, I1.3-GND, I44.G, LS.1, LS.3, M0.8, M1.8, M2.8, M3.8, M4.8, M5.14, M5.8, U$2.1, U$3.1, U$4.1, U$5.1; no longer C16.1, C17.1, C25.2, C26.2, U$1.G, U$14.1, U$14.3, U10.14, U10.8, U5.8, U6.8, U7.8, U8.8, U9.8
- net K00: now also M0.15; no longer U5.15
- net K01: now also M0.1; no longer U5.1
- net K02: now also M0.2; no longer U5.2
- net K03: now also M0.3; no longer U5.3
- net K04: now also M0.4; no longer U5.4
- net K05: now also M0.5; no longer U5.5
- net K06: now also M0.6; no longer U5.6
- net K07: now also M0.7; no longer U5.7
- net K10: now also M1.15; no longer U6.15
- net K11: now also M1.1; no longer U6.1
- net K12: now also M1.2; no longer U6.2
- net K13: now also M1.3; no longer U6.3
- net K14: now also M1.4; no longer U6.4
- net K15: now also M1.5; no longer U6.5
- net K16: now also M1.6; no longer U6.6
- net K17: now also M1.7; no longer U6.7
- net K20: now also M2.15; no longer U7.15
- net K21: now also M2.1; no longer U7.1
- net K22: now also M2.2; no longer U7.2
- net K23: now also M2.3; no longer U7.3
- net K24: now also M2.4; no longer U7.4
- net K25: now also M2.5; no longer U7.5
- net K26: now also M2.6; no longer U7.6
- net K27: now also M2.7; no longer U7.7
- net K30: now also M3.15; no longer U8.15
- net K31: now also M3.1; no longer U8.1
- net K32: now also M3.2; no longer U8.2
- net K33: now also M3.3; no longer U8.3
- net K34: now also M3.4; no longer U8.4
- net K35: now also M3.5; no longer U8.5
- net K36: now also M3.6; no longer U8.6
- net K37: now also M3.7; no longer U8.7
- net K40: now also M4.15; no longer U9.15
- net K41: now also M4.1; no longer U9.1
- net K42: now also M4.2; no longer U9.2
- net K43: now also M4.3; no longer U9.3
- net K44: now also M4.4; no longer U9.4
- net K45: now also M4.5; no longer U9.5
- net K46: now also M4.6; no longer U9.6
- net K47: now also M4.7; no longer U9.7
- net K50: now also M5.15; no longer U10.15
- net K51: now also M5.1; no longer U10.1
- net K52: now also M5.2; no longer U10.2
- net K53: now also M5.3; no longer U10.3
- net K54: now also M5.4; no longer U10.4
- net K55: now also M5.5; no longer U10.5
- net K56: now also M5.6; no longer U10.6
- net K57: now also M5.7; no longer U10.7
- net LED1ST: now also LS.2; no longer U$14.2
- net MATRIX_1_2: now also M0.14, M1.9; no longer U5.14, U6.9
- net MATRIX_2_3: now also M1.14, M2.9; no longer U6.14, U7.9
- net MATRIX_3_4: now also M2.14, M3.9; no longer U7.14, U8.9
- net MATRIX_4_5: now also M3.14, M4.9; no longer U8.14, U9.9
- net MATRIX_5_6: now also M4.14, M5.9; no longer U10.9, U9.14
- net MATRIX_CS: now also M0.10, M1.10, M2.10, M3.10, M4.10, M5.10, U$2.5, U$3.5; no longer U10.10, U5.10, U6.10, U7.10, U8.10, U9.10
- net MATRIX_LATCH: now also M0.12, M0.13, M1.12, M1.13, M2.12, M2.13, M3.12, M3.13, M4.12, M4.13, M5.12, M5.13; no longer U10.12, U10.13, U5.12, U5.13, U6.12, U6.13, U7.12, U7.13, U8.12, U8.13, U9.12, U9.13
- net N$22: now also I20.2-DOUT, I21.4-DIN; no longer I10.4-DIN, I31.2-DOUT
- net N$3: now also I10.4-DIN; no longer U$1.D
- net N$66: now also LS.4; no longer C44.1, U$14.4
- net OSC32_I: now also C25.2; no longer C16.2
- net OSC32_O: now also C26.2; no longer C17.2
- net SPI_MISO: now also M0.9, U$2.4, U$3.4; no longer U5.9
- net SPI_MOSI: now also U$2.3, U$3.3
- net SPI_SCK: now also M0.11, M1.11, M2.11, M3.11, M4.11, M5.11; no longer U10.11, U5.11, U6.11, U7.11, U8.11, U9.11
- net VCC_1: now also C16.1, C17.1, C20.1; no longer C23.1, C25.1, C26.1
- net VCC_2: now also C23.1, M0.16, M1.16, M2.16, M3.16, M4.16, M5.16, U$2.2, U$3.2; no longer C20.1, U10.16, U5.16, U6.16, U7.16, U8.16, U9.16
Routing:
- net USB_DP: track 0.00 -> 8.66 mm
- net USB_DN: track 0.00 -> 8.45 mm
- net VCC_1: track 0.00 -> 1.72 mm
Other:
- board size 227.6 x 74.2 mm -> 260 x 80 mm
- board text added: "RESET"
- board text added: "pwr"
