File: EAGLE/vr42/vr42-revA.sch (EAGLE design)
At the start: 1 part

Commit message: sch
Parts:
- removed U$1: STM32F4R_64PIN_FOXCAR, stm32f4:STM32F4R_64PIN_FOXCAR
Changed lines of the file:
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@@
 <layer number="59" name="tCarbon" color="7" fill="1" visible="no" active="no"/>
 <layer number="60" name="bCarbon" color="7" fill="1" visible="no" active="no"/>
+<layer number="61" name="stand" color="7" fill="1" visible="no" active="no"/>
 <layer number="88" name="SimResults" color="9" fill="1" visible="yes" active="yes"/>
 <layer number="89" name="SimProbes" color="9" fill="1" visible="yes" active="yes"/>
@@
 <layer number="146" name="DrillLegend_01-20" color="7" fill="1" visible="no" active="no"/>
 <layer number="147" name="PIN_NUMBER" color="7" fill="1" visible="no" active="no"/>
+<layer number="148" name="mDocument" color="7" fill="1" visible="yes" active="yes"/>
 <layer number="149" name="DrillLegend_02-15" color="7" fill="1" visible="no" active="no"/>
 <layer number="150" name="Notes" color="7" fill="1" visible="no" active="no"/>
@@
 <layer number="154" name="FabDoc2" color="7" fill="1" visible="no" active="no"/>
 <layer number="155" name="FabDoc3" color="7" fill="1" visible="no" active="no"/>
+<layer number="160" name="O_Dim" color="7" fill="1" visible="no" active="yes"/>
 <layer number="166" name="AntennaArea" color="7" fill="1" visible="no" active="no"/>
 <layer number="168" name="4mmHeightArea" color="7" fill="1" visible="no" active="no"/>
@@
 <parts>
 <part name="FRAME1" library="SparkFun-Aesthetics" deviceset="FRAME-A4L" device=""/>
-<part name="U$1" library="stm32f4" deviceset="STM32F4R_64PIN_FOXCAR" device=""/>
 </parts>
 <sheets>
@@
 <attribute name="DESIGNER" x="226.26" y="6.35" size="2.54" layer="94" font="vector"/>
 </instance>
-<instance part="U$1" gate="G$1" x="129.54" y="83.82" smashed="yes"/>
 </instances>
 <busses>
@@
 </schematic>
 </drawing>
-<compatibility>
-<note version="6.3" minversion="6.2.2" severity="warning">
-Since Version 6.2.2 text objects can contain more than one line,
-which will not be processed correctly with this version.
-</note>
-</compatibility>
 </eagle>

Commit message: wip
Parts:
- added C1, C2: 2.2uF, rcl:C-EUC0603
- added C10, C11: 9pF, rcl:C-EUC0603
- added C12, C13, C14, C15, C25, C26, C8: 0.1uF, rcl:C-EUC0603
- added C16, C17: 2.2pF, rcl:C-EUC0603
- added C18, C19: 12pF, rcl:C-EUC0603
- added C20, C21, C28: 100nF, SparkFun-Capacitors:0.1UF-0603-25V-5%
- added C22, C23: 22uF, SparkFun-Capacitors:0.22UF-0603-25V-10%
- added C24: 4.7uF, SparkFun-Capacitors:1.0NF/1000PF-0603-50V-10%
- added C27, C3, C4, C5, C6, C7: 100nF, rcl:C-EUC0603
- added C29, C32, C33, C34, C35, C36, C37: (no value), rcl:C-EUC0603
- added C30: 1uF, rcl:C-EUC0805
- added C31: 100nF, rcl:C-EUC0805
- added C9: 1uF, rcl:C-EUC0603
- added D00: B5819W SL, jlcpcb_basic_parts:1N5819WS
- added D107: BLUE, SparkFun-LED:LED-BLUE0603
- added D201, D202: 1N4148, adafruit:DIODESOT23_REFLOW
- added H_RS1, H_RS2: MX-STABS-200U, ts_keyboards:MX-STABS-200U
- added J1: (no value), SparkFun-Connectors:CONN_02
- added JI2C, JPWM: (no value), SparkFun-Connectors:CONN_04
- added JSPI: DNP, SparkFun-Connectors:AVR_SPI_PROG_3X2NS
- added JSPI@2: (no value), SparkFun-Connectors:CONN_01
- added JTAG: DNP, SparkFun-Connectors:CONN_05X2NO_SILK
- added L1: 10uH ±10%, rcl:L-USL3225M
- added LM1117: AMS1117-3.3, SparkFun-IC-Power:V_REG_LM1117SOT223
- added Q2: DMG2305UX-7, SparkFun-DiscreteSemi:MOSFET_PCH-DMG2305UX-7
- added R1: 820R, rcl:R-EU_R0603
- added R10, R9: 100K, rcl:R-EU_R0603
- added R11, R12, R4: 1K, rcl:R-EU_R0603
- added R13, R7: 10K, rcl:R-EU_R0603
- added R2: 12K, rcl:R-EU_R0603
- added R3: 1M, rcl:R-EU_R0603
- added R5, R6: 22R, rcl:R-EU_R0603
- added R8: /DNP/, rcl:R-EU_R0603
- added S1: Reset, SparkFun-Switches:MOMENTARY-SWITCH-SPST-SMD-5.2-TALL-REDUNDANT
- added SW_A, SW_B, SW_BSP, SW_C, SW_D, SW_DEL, SW_DN, SW_E, SW_ENT, SW_ESC, SW_F, SW_G, SW_H, SW_I, SW_J, SW_K, SW_L, SW_LA, SW_LC, SW_LF, SW_LS, SW_LW, SW_M, SW_N, SW_O, SW_P, SW_Q, SW_R, SW_RS, SW_RT, SW_S, SW_SPC_1, SW_SPC_2, SW_T, SW_TAB, SW_U, SW_UP, SW_V, SW_W, SW_X, SW_Y, SW_Z: MX-5-PIN-HOTSWAP-PAD, ts_keyboards:MX-5-PIN-HOTSWAP-PAD
- added U1: STM32F405RGT6, st:STM32F405RGT6
- added U2: USB3300-EZK, ts_kb_mcu:USB3300-EZK
- added U3: TS3USB221A-Q1, ts_kb_mcu:TS3USB221A-Q1
- added U5: M25C, ts_kb_mcu:M25C
- added UDB1: (no value), ts_keyboards:UBD-S1_C4
- added UDB2: (no value), ts_keyboards:UBD-C3
- added Y1: 32.768kHz ±20ppm 6pF, SparkFun-Clocks:CRYSTAL-32.768KHZSMD-3.2X1.5
- added Y2: 25MHz 9pF, SparkFun-Clocks:CRYSTAL-24MHZ"
- added Y3: 24MHz, SparkFun-Clocks:CRYSTAL-24MHZ"
Connections:
- new net !BOOT: C31.1, D202.A, Q2.G, R9.1
- new net !RESET: C29.2, D201.A, R8.1, U1B.NRST
- new net AUX_CS: JSPI.5
- new net AUX_DC: JSPI@2.1
- new net BOOT0: Q2.D, R10.1, U1B.BOOT0
- new net BOOT1: R7.2, U1B.PB2/BOOT1
- new net CK/DATA/PWM: JPWM.3
- new net EE_CS: U5.!CS
- new net GND: C1.2, C10.2, C11.2, C12.2, C13.2, C14.2, C15.2, C16.1, C17.1, C18.1, C19.1, C2.2, C20.2, C21.2, C22.2, C23.2, C24.2, C25.2, C26.2, C27.2, C28.2, C29.1, C3.2, C30.2, C31.2, C32.2, C34.2, C35.2, C36.2, C37.2, C4.2, C5.2, C6.2, C7.2, C8.2, C9.2, J1.1, JI2C.4, JPWM.4, JSPI.6, JTAG.3, JTAG.5, JTAG.9, LM1117.ADJ, R10.2, R13.1, R2.2, R7.1, S1.1, U1A.VSS, U1A.VSSA, U1A.VSS_2, U2.EPAD, U2.GND_1, U2.GND_2, U2.RESET, U3.!OE, U3.GND, U5.GND, UDB1.GND, UDB1.M, UDB2.GND, UDB2.M
- new net HS_ULPI_CK: U1B.PA5, U2.CLKOUT
- new net HS_ULPI_D0: U1B.PA3, U2.DATA0
- new net HS_ULPI_D1: U1B.PB0, U2.DATA1
- new net HS_ULPI_D2: U1B.PB1, U2.DATA2
- new net HS_ULPI_D3: U1B.PB10, U2.DATA3
- new net HS_ULPI_D4: U1B.PB11, U2.DATA4
- new net HS_ULPI_D5: U1B.PB12, U2.DATA5
- new net HS_ULPI_D6: U1B.PB13, U2.DATA6
- new net HS_ULPI_D7: U1B.PB5, U2.DATA7
- new net HS_ULPI_DIR: U1B.PC2, U2.DIR
- new net HS_ULPI_NXT: U1B.PC3, U2.NXT
- new net HS_ULPI_STP: U1B.PC0, U2.STP
- new net I2C_SCL: R11.1, U1B.PB6
- new net I2C_SDA: R12.1, U1B.PB7
- new net J_RST: JTAG.10
- new net J_TCK: JTAG.4
- new net J_TDI: JTAG.8
- new net J_TDO: JTAG.6
- new net J_TMS: JTAG.2
- new net K00: SW_ESC.P
- new net K01: SW_Q.P
- new net K02: SW_W.P
- new net K03: SW_E.P
- new net K04: SW_TAB.P
- new net K05: SW_A.P
- new net K06: SW_S.P
- new net K07: SW_D.P
- new net K10: SW_R.P
- new net K11: SW_T.P
- new net K12: SW_Y.P
- new net K13: SW_U.P
- new net K14: SW_F.P
- new net K15: SW_G.P
- new net K16: SW_H.P
- new net K17: SW_J.P
- new net K20: SW_I.P
- new net K21: SW_O.P
- new net K22: SW_P.P
- new net K23: SW_BSP.P
- new net K24: SW_K.P
- new net K25: SW_L.P
- new net K26: SW_ENT.P
- new net K30: SW_LS.P
- new net K31: SW_Z.P
- new net K32: SW_X.P
- new net K34: SW_LC.P
- new net K35: SW_LW.P
- new net K36: SW_LA.P
- new net K40: SW_C.P
- new net K41: SW_V.P
- new net K42: SW_B.P
- new net K43: SW_N.P
- new net K44: SW_SPC_1.P
- new net K45: SW_SPC_2.P
- new net K50: SW_M.P
- new net K51: SW_RS.P
- new net K52: SW_UP.P
- new net K53: SW_DEL.P
- new net K54: SW_LF.P
- new net K55: SW_DN.P
- new net K56: SW_RT.P
- new net LED: D107.C
- new net MISO: JSPI.1
- new net MOSI: JSPI.4
- new net N$1: C1.1, U1A.VCAP_2
- new net N$10: R2.1, U2.RBIAS
- new net N$11: U1B.PA8
- new net N$12: U1B.PA9
- new net N$140: R5.2, U1B.PA11
- new net N$141: R6.2, U1B.PA12
- new net N$145: D107.A, R4.2
- new net N$16: U1B.PA13
- new net N$17: U1B.PA14
- new net N$18: U1B.PA15
- new net N$19: C8.1, U2.VDDA1.8
- new net N$2: C2.1, U1A.VCAP_1
- new net N$22: U1B.PB4
- new net N$26: U1B.PB8
- new net N$28: U1B.PB9
- new net N$3: U1B.PA0/WKUP
- new net N$33: U1B.PB14
- new net N$34: U1B.PB15
- new net N$36: U1B.PC1
- new net N$39: U1B.PC4
- new net N$4: U1B.PA1
- new net N$40: U1B.PC5
- new net N$41: U1B.PC6
- new net N$42: U1B.PC7
- new net N$43: U1B.PC8
- new net N$44: U1B.PC9
- new net N$48: U1B.PC13
- new net N$5: U1B.PA2
- new net N$51: U1B.PD2
- new net N$7: U1B.PA4
- new net N$9: R1.2, U2.VBUS
- new net OSC32_I: C16.2, U1B.PC14/OSC32_IN, Y1.2
- new net OSC32_O: C17.2, U1B.PC15/OSC32_OUT, Y1.1
- new net OSC_I: C18.2, U1B.PH0/OSC_IN, Y2.2
- new net OSC_O: C19.2, U1B.PH1/OSC_OUT, Y2.1
- new net RESET: D201.C, D202.C, J1.2, S1.2
- new net SCK: JSPI.3
- new net SCL: JI2C.1
- new net SDA: JI2C.2
- new net SPI_MISO: U1B.PA6, U5.DO
- new net SPI_MOSI: U1B.PA7, U5.DIO
- new net SPI_SCK: U1B.PB3, U5.CLK
- new net ULPI_1V8: C12.1, C13.1, U2.VDD1.8_1, U2.VDD1.8_2
- new net ULPI_XI: C11.1, R3.2, U2.XI, Y3.2
- new net ULPI_XO: C10.1, R3.1, U2.XO, Y3.1
- new net USART_CK: U1B.PC12
- new net USART_RX: U1B.PC11
- new net USART_TX: U1B.PC10
- new net USB1_DN: R5.1, U3.1D-
- new net USB1_DP: R6.1, U3.1D+
- new net USB2_DN: U2.DM, U3.2D-
- new net USB2_DP: U2.DP, U3.2D+
- new net USB_DN: U3.D-, UDB1.DN, UDB2.DN
- new net USB_DP: U3.D+, UDB1.DP, UDB2.DP
- new net USB_SELECT: R13.2, U1B.PA10, U3.S
- new net VCC_1: C14.1, C15.1, C21.1, C23.1, C25.1, C26.1, C30.1, C9.1, D00.C, JPWM.1, LM1117.IN, R1.1, U2.REG_EN, U2.VDD3.3_1, U2.VDD3.3_2, U2.VDD3.3_3, U2.VDD3.3_4, UDB1.VCC, UDB2.VCC
- new net VCC_2: C20.1, C22.1, C24.1, C27.1, C28.1, C32.1, C34.1, C35.1, C36.1, C37.1, C4.1, C5.1, C6.1, C7.1, D00.A, JI2C.3, JPWM.2, JSPI.2, JTAG.1, L1.1, LM1117.OUT, Q2.S, R11.2, R12.2, R4.1, R8.2, R9.2, SW_A.S, SW_B.S, SW_BSP.S, SW_C.S, SW_D.S, SW_DEL.S, SW_DN.S, SW_E.S, SW_ENT.S, SW_ESC.S, SW_F.S, SW_G.S, SW_H.S, SW_I.S, SW_J.S, SW_K.S, SW_L.S, SW_LA.S, SW_LC.S, SW_LF.S, SW_LS.S, SW_LW.S, SW_M.S, SW_N.S, SW_O.S, SW_P.S, SW_Q.S, SW_R.S, SW_RS.S, SW_RT.S, SW_S.S, SW_SPC_1.S, SW_SPC_2.S, SW_T.S, SW_TAB.S, SW_U.S, SW_UP.S, SW_V.S, SW_W.S, SW_X.S, SW_Y.S, SW_Z.S, U1A.VBAT, U1A.VDD, U1A.VDD_2, U1A.VDD_3, U1A.VDD_4, U3.VCC, U5.!HLD, U5.!WP, U5.VCC
- new net VDDA: C3.1, L1.2, U1A.VDDA
Other:
- note added: "!RESET"
- note added: "** NEW ** Unified Daughter Board (C4) Conn."
- note added: "5V to 3V3 Power Circuit"
- note added: "BOOT0 Inversion"
- note added: "BOOT1"
- note added: "DNP Unified Daughter Board (C3) Conn. (Legacy)"
- note added: "I2C Pull-ups"
- note added: "SPI EEPROM (Optional)"
- note added: "Status LED"
- note added: "U1 Clocks"
- note added: "U2 1.8V Caps"
- note added: "U2 Clock"
- note added: "U2 VDD Caps"
- note added: "U3 VDD Cap"

Commit message: .
Parts:
- removed JI2C, JPWM: (no value), SparkFun-Connectors:CONN_04
- added C38, C39, C40, C41, C42, C43: 100nF, SparkFun-Capacitors:0.1UF-0603-25V-5%
- added C44, C45, C46, C47, C48, C49, C50: 100nF, rcl:C-EUC0603
- added JSPI@3: (no value), SparkFun-Connectors:CONN_01
- added LED_A, LED_B, LED_BSP, LED_C, LED_D, LED_DEL, LED_DN, LED_E, LED_ENT, LED_ESC, LED_F, LED_G, LED_H, LED_I, LED_J, LED_K, LED_L, LED_LA, LED_LC, LED_LF, LED_LS, LED_LW, LED_M, LED_N, LED_O, LED_P, LED_Q, LED_R, LED_RS, LED_RT, LED_S, LED_SPC_1@1, LED_SPC_1@2, LED_SPC_1@3, LED_SPC_2@1, LED_SPC_2@2, LED_SPC_2@3, LED_T, LED_TAB, LED_U, LED_UP, LED_V, LED_W, LED_X, LED_Y, LED_Z: SK6812-E-REVERSE, ts_keyboards:SK6812-E-REVERSE
- added Q1: 2N7002, adafruit:MOSFET-NREFLOW
- added R14, R15, R16, R17, R18, R19, R20, R21, R22, R23, R24, R25: 10K, ts_keyboards:R-EU-4
- added R26, R28, R29: 5.1K, rcl:R-EU_R0603
- added R27: 75K, rcl:R-EU_R0603
- added U$1: ARGB, __temp_to_delete:ARGB
- added U$14: 74AHCT1G125GW, ts_keyboards:74AHCT1G125GW
- added U10, U6, U7, U8, U9: 74HC589A_DT, __untitled:74HC589A_DT
- added U4: TPS2553DBVR-1, __untitled:TPS2553DBVR-1
- added U4X: M25C, ts_kb_mcu:M25C
- C12, C13, C8: value 0.1uF -> 4.7uF
- C29, C32, C33, C34, C35, C36, C37: value (none) -> 100nF
- R11: value 1K -> 220
- R12: value 1K -> 470
- R3: value 1M -> 10M
- U5: value M25C -> 74HC589A_DT; device ts_kb_mcu:M25C -> __untitled:74HC589A_DT
Connections:
- net N$48 renamed ANTI_TAMP
- removed net CK/DATA/PWM: JPWM.3
- removed net I2C_SCL: R11.1, U1B.PB6
- removed net I2C_SDA: R12.1, U1B.PB7
- removed net J_RST: JTAG.10
- removed net J_TCK: JTAG.4
- removed net J_TDI: JTAG.8
- removed net J_TDO: JTAG.6
- removed net J_TMS: JTAG.2
- removed net MISO: JSPI.1
- removed net MOSI: JSPI.4
- removed net N$43: U1B.PC8
- removed net N$44: U1B.PC9
- removed net SCK: JSPI.3
- removed net SCL: JI2C.1
- removed net SDA: JI2C.2
- removed net USART_CK: U1B.PC12
- removed net USART_RX: U1B.PC11
- removed net USART_TX: U1B.PC10
- new net !ARGB_FAULT: R28.2, U1B.PD2, U4.!FAULT
- new net ARGB_D: R11.2, U1B.PB7
- new net ARGB_EN: R29.1, U1B.PB6, U4.EN
- new net AUX_RST: JSPI@3.1, U1B.PB15
- new net JTCK: JTAG.4, U1B.PA14
- new net JTDI: JTAG.8, U1B.PA15
- new net JTDO: JTAG.6, U1B.PB3
- new net JTMS: JTAG.2, U1B.PA13
- new net JTRST: JTAG.10, U1B.PB4
- new net K27: R18.1, U7.H
- new net K33: R21.5, U8.D
- new net K37: R20.1, U8.H
- new net K46: R22.2, U9.G
- new net K47: R22.1, U9.H
- new net K57: R24.1, U10.H
- new net LED1ST: R11.1, U$14.A_DIN
- new net MATRIX_1_2: U5.SA, U6.QH
- new net MATRIX_2_3: U6.SA, U7.QH
- new net MATRIX_3_4: U7.SA, U8.QH
- new net MATRIX_4_5: U8.SA, U9.QH
- new net MATRIX_5_6: U10.QH, U9.SA
- new net MATRIX_CS: Q1.G, U10.OE/!CS, U1B.PC4, U5.OE/!CS, U6.OE/!CS, U7.OE/!CS, U8.OE/!CS, U9.OE/!CS
- new net MATRIX_LATCH: Q1.D, R26.1, U10.LATCH, U10.SS/!PL, U5.LATCH, U5.SS/!PL, U6.LATCH, U6.SS/!PL, U7.LATCH, U7.SS/!PL, U8.LATCH, U8.SS/!PL, U9.LATCH, U9.SS/!PL
- new net N$13: LED_I.4_DIN, LED_U.2_DOUT
- new net N$14: LED_J.4_DIN, LED_K.2_DOUT
- new net N$15: LED_H.4_DIN, LED_J.2_DOUT
- new net N$20: LED_A.4_DIN, LED_S.2_DOUT
- new net N$21: LED_A.2_DOUT, LED_TAB.4_DIN
- new net N$23: LED_LS.2_DOUT, LED_Z.4_DIN
- new net N$24: LED_X.4_DIN, LED_Z.2_DOUT
- new net N$25: LED_C.4_DIN, LED_X.2_DOUT
- new net N$27: LED_B.4_DIN, LED_V.2_DOUT
- new net N$29: LED_M.4_DIN, LED_N.2_DOUT
- new net N$30: LED_O.4_DIN
- new net N$31: LED_SPC_2@1.4_DIN, LED_SPC_2@2.2_DOUT
- new net N$32: LED_SPC_1@3.4_DIN, LED_SPC_2@1.2_DOUT
- new net N$35: LED_LA.4_DIN, LED_SPC_1@1.2_DOUT
- new net N$37: LED_LC.4_DIN, LED_LW.2_DOUT
- new net N$38: R27.2, U4.ILIM
- new net N$46: LED_DN.4_DIN, LED_RT.2_DOUT
- new net N$47: LED_BSP.4_DIN, LED_P.2_DOUT
- new net N$48: LED_ENT.2_DOUT, LED_L.4_DIN
- new net N$49: LED_K.4_DIN, LED_L.2_DOUT
- new net N$50: LED_DN.2_DOUT, LED_LF.4_DIN
- new net N$52: LED_SPC_2@2.4_DIN, LED_SPC_2@3.2_DOUT
- new net N$54: LED_M.2_DOUT, LED_RS.4_DIN
- new net N$55: LED_RS.2_DOUT, LED_UP.4_DIN
- new net N$6: LED_E.4_DIN, LED_W.2_DOUT
- new net N$61: LED_DEL.2_DOUT, LED_RT.4_DIN
- new net N$66: C44.1, R12.2, U$14.Y_DOUT
- new net N$8: LED_R.2_DOUT, LED_T.4_DIN
- new net SK6803: LED_ESC.4_DIN, R12.1
- new net SK6803_PWR: C46.1, C47.1, C48.1, C49.1, C50.1, LED_A.1_VDD, LED_B.1_VDD, LED_BSP.1_VDD, LED_C.1_VDD, LED_D.1_VDD, LED_DEL.1_VDD, LED_DN.1_VDD, LED_E.1_VDD, LED_ENT.1_VDD, LED_ESC.1_VDD, LED_F.1_VDD, LED_G.1_VDD, LED_H.1_VDD, LED_I.1_VDD, LED_J.1_VDD, LED_K.1_VDD, LED_L.1_VDD, LED_LA.1_VDD, LED_LC.1_VDD, LED_LF.1_VDD, LED_LS.1_VDD, LED_LW.1_VDD, LED_M.1_VDD, LED_N.1_VDD, LED_O.1_VDD, LED_P.1_VDD, LED_Q.1_VDD, LED_R.1_VDD, LED_RS.1_VDD, LED_RT.1_VDD, LED_S.1_VDD, LED_SPC_1@1.1_VDD, LED_SPC_1@2.1_VDD, LED_SPC_1@3.1_VDD, LED_SPC_2@1.1_VDD, LED_SPC_2@2.1_VDD, LED_SPC_2@3.1_VDD, LED_T.1_VDD, LED_TAB.1_VDD, LED_U.1_VDD, LED_UP.1_VDD, LED_V.1_VDD, LED_W.1_VDD, LED_X.1_VDD, LED_Y.1_VDD, LED_Z.1_VDD, U$1.V, U$14.5_VCC, U4.OUT
- net !RESET: now also C29.1; no longer C29.2
- net AUX_CS: now also U1B.PA2
- net AUX_DC: now also U1B.PB14
- net EE_CS: now also U1B.PA1, U4X.!CS; no longer U5.!CS
- net GND: now also C29.2, C33.2, C38.2, C39.2, C40.2, C41.2, C42.2, C43.2, C44.2, C45.2, C46.2, C47.2, C48.2, C49.2, C50.2, LED_A.3_GND, LED_B.3_GND, LED_BSP.3_GND, LED_C.3_GND, LED_D.3_GND, LED_DEL.3_GND, LED_DN.3_GND, LED_E.3_GND, LED_ENT.3_GND, LED_ESC.3_GND, LED_F.3_GND, LED_G.3_GND, LED_H.3_GND, LED_I.3_GND, LED_J.3_GND, LED_K.3_GND, LED_L.3_GND, LED_LA.3_GND, LED_LC.3_GND, LED_LF.3_GND, LED_LS.3_GND, LED_LW.3_GND, LED_M.3_GND, LED_N.3_GND, LED_O.3_GND, LED_P.3_GND, LED_Q.3_GND, LED_R.3_GND, LED_RS.3_GND, LED_RT.3_GND, LED_S.3_GND, LED_SPC_1@1.3_GND, LED_SPC_1@2.3_GND, LED_SPC_1@3.3_GND, LED_SPC_2@1.3_GND, LED_SPC_2@2.3_GND, LED_SPC_2@3.3_GND, LED_T.3_GND, LED_TAB.3_GND, LED_U.3_GND, LED_UP.3_GND, LED_V.3_GND, LED_W.3_GND, LED_X.3_GND, LED_Y.3_GND, LED_Z.3_GND, Q1.S, R14.5, R14.6, R14.7, R14.8, R15.1, R15.2, R15.3, R15.4, R16.5, R16.6, R16.7, R16.8, R17.1, R17.2, R17.3, R17.4, R18.5, R18.6, R18.7, R18.8, R19.1, R19.2, R19.3, R19.4, R20.5, R20.6, R20.7, R20.8, R21.1, R21.2, R21.3, R21.4, R22.5, R22.6, R22.7, R22.8, R23.1, R23.2, R23.3, R23.4, R24.5, R24.6, R24.7, R24.8, R25.1, R25.2, R25.3, R25.4, R27.1, R29.2, U$1.G, U$14.!OE, U$14.3_GND, U10.GND, U10.SA, U4.GND, U4X.GND, U6.GND, U7.GND, U8.GND, U9.GND; no longer C29.1, JI2C.4, JPWM.4
- net K00: now also R15.8, U5.A
- net K01: now also R15.7, U5.B
- net K02: now also R15.6, U5.C
- net K03: now also R15.5, U5.D
- net K04: now also R14.4, U5.E
- net K05: now also R14.3, U5.F
- net K06: now also R14.2, U5.G
- net K07: now also R14.1, U5.H
- net K10: now also R17.8, U6.A
- net K11: now also R17.7, U6.B
- net K12: now also R17.6, U6.C
- net K13: now also R17.5, U6.D
- net K14: now also R16.4, U6.E
- net K15: now also R16.3, U6.F
- net K16: now also R16.2, U6.G
- net K17: now also R16.1, U6.H
- net K20: now also R19.8, U7.A
- net K21: now also R19.7, U7.B
- net K22: now also R19.6, U7.C
- net K23: now also R19.5, U7.D
- net K24: now also R18.4, U7.E
- net K25: now also R18.3, U7.F
- net K26: now also R18.2, U7.G
- net K30: now also R21.8, U8.A
- net K31: now also R21.7, U8.B
- net K32: now also R21.6, U8.C
- net K34: now also R20.4, U8.E
- net K35: now also R20.3, U8.F
- net K36: now also R20.2, U8.G
- net K40: now also R23.8, U9.A
- net K41: now also R23.7, U9.B
- net K42: now also R23.6, U9.C
- net K43: now also R23.5, U9.D
- net K44: now also R22.4, U9.E
- net K45: now also R22.3, U9.F
- net K50: now also R25.8, U10.A
- net K51: now also R25.7, U10.B
- net K52: now also R25.6, U10.C
- net K53: now also R25.5, U10.D
- net K54: now also R24.4, U10.E
- net K55: now also R24.3, U10.F
- net K56: now also R24.2, U10.G
- net LED: now also U1B.PB8
- net N$11: now also LED_T.2_DOUT, LED_Y.4_DIN; no longer U1B.PA8
- net N$12: now also LED_U.4_DIN, LED_Y.2_DOUT; no longer U1B.PA9
- net N$16: now also LED_G.4_DIN, LED_H.2_DOUT; no longer U1B.PA13
- net N$17: now also LED_F.4_DIN, LED_G.2_DOUT; no longer U1B.PA14
- net N$18: now also LED_D.4_DIN, LED_F.2_DOUT; no longer U1B.PA15
- net N$22: now also LED_LS.4_DIN, LED_TAB.2_DOUT; no longer U1B.PB4
- net N$26: now also LED_C.2_DOUT, LED_V.4_DIN; no longer U1B.PB8
- net N$28: now also LED_B.2_DOUT, LED_N.4_DIN; no longer U1B.PB9
- net N$3: now also LED_LC.2_DOUT, U$1.D; no longer U1B.PA0/WKUP
- net N$33: now also LED_SPC_1@2.4_DIN, LED_SPC_1@3.2_DOUT; no longer U1B.PB14
- net N$34: now also LED_SPC_1@1.4_DIN, LED_SPC_1@2.2_DOUT; no longer U1B.PB15
- net N$36: now also LED_LA.2_DOUT, LED_LW.4_DIN; no longer U1B.PC1
- net N$39: now also LED_BSP.2_DOUT, LED_ENT.4_DIN; no longer U1B.PC4
- net N$4: now also LED_ESC.2_DOUT, LED_Q.4_DIN; no longer U1B.PA1
- net N$40: now also LED_DEL.4_DIN, LED_UP.2_DOUT; no longer U1B.PC5
- net N$41: now also LED_O.2_DOUT, LED_P.4_DIN; no longer U1B.PC6
- net N$42: now also LED_D.2_DOUT, LED_S.4_DIN; no longer U1B.PC7
- net N$5: now also LED_Q.2_DOUT, LED_W.4_DIN; no longer U1B.PA2
- net N$51: now also LED_LF.2_DOUT, LED_SPC_2@3.4_DIN; no longer U1B.PD2
- net N$7: now also LED_E.2_DOUT, LED_R.4_DIN; no longer U1B.PA4
- net SPI_MISO: now also JSPI.1, U1B.PC11, U4X.DO, U5.QH; no longer U1B.PA6, U5.DO
- net SPI_MOSI: now also JSPI.4, U1B.PC12, U4X.DIO; no longer U1B.PA7, U5.DIO
- net SPI_SCK: now also JSPI.3, U10.SC/SCK, U1B.PC10, U4X.CLK, U5.SC/SCK, U6.SC/SCK, U7.SC/SCK, U8.SC/SCK, U9.SC/SCK; no longer U1B.PB3, U5.CLK
- net USB_SELECT: now also U1B.PB9; no longer U1B.PA10
- net VCC_1: now also C45.1, R28.1, U4.IN; no longer JPWM.1
- net VCC_2: now also C33.1, C38.1, C39.1, C40.1, C41.1, C42.1, C43.1, R26.2, U10.VCC, U4X.!HLD, U4X.!WP, U4X.VCC, U6.VCC, U7.VCC, U8.VCC, U9.VCC; no longer JI2C.3, JPWM.2, R11.2, R12.2, U5.!HLD, U5.!WP
Other:
- note added: "74HC589A VDD Caps (Place near each VCC pin)"
- note added: "USB = 500mA Max, Rlim = 75K = 74.25 @ 1% = 319mA - 401mA range"
- note removed: "I2C Pull-ups"

Commit message: .
Parts:
- removed LED_DN, LED_LF, LED_RT, LED_SPC_2@3: SK6812-E-REVERSE, ts_keyboards:SK6812-E-REVERSE
- renumbered H_RS1 to H_SPC_1, H_RS2 to H_SPC_2, LED_A to Z22, LED_B to Z29, LED_BSP to Z12, LED_C to Z27, LED_D to Z20, LED_DEL to Z34, LED_E to Z4, LED_ENT to Z13, LED_ESC to Z1, LED_F to Z19, LED_G to Z18, LED_H to Z17, LED_I to Z9, LED_J to Z16, LED_K to Z15, LED_L to Z14, LED_LA to Z40, LED_LC to Z42, LED_LS to Z24, LED_LW to Z41, LED_M to Z31, LED_N to Z30, LED_O to Z10, LED_P to Z11, LED_Q to Z2, LED_R to Z5, LED_RS to Z32, LED_S to Z21, LED_SPC_1@1 to Z39, LED_SPC_1@2 to Z38, LED_SPC_1@3 to Z37, LED_SPC_2@1 to Z36, LED_SPC_2@2 to Z35, LED_T to Z6, LED_TAB to Z23, LED_U to Z8, LED_UP to Z33, LED_V to Z28, LED_W to Z3, LED_X to Z26, LED_Y to Z7, LED_Z to Z25
Connections:
- removed net N$46 (its old number): LED_DN.4_DIN, LED_RT.2_DOUT
- removed net N$50 (its old number): LED_DN.2_DOUT, LED_LF.4_DIN
- removed net N$51 (its old number): LED_LF.2_DOUT, LED_SPC_2@3.4_DIN
- removed net N$52 (its old number): LED_SPC_2@3.2_DOUT, Z35.4_DIN
- net GND: no longer LED_DN.3_GND, LED_LF.3_GND, LED_RT.3_GND, LED_SPC_2@3.3_GND
- net N$61: now also Z35.4_DIN; no longer LED_RT.4_DIN
- net SK6803_PWR: no longer LED_DN.1_VDD, LED_LF.1_VDD, LED_RT.1_VDD, LED_SPC_2@3.1_VDD

Commit message: .
Parts:
- removed U$14: 74AHCT1G125GW, ts_keyboards:74AHCT1G125GW
- added I1: SK6812-E-REVERSE, ts_keyboards:SK6812-E-REVERSE
- added I44: ARGB, __temp_to_delete:ARGB
- added LS: 74AHCT1G125GW, ts_keyboards:74AHCT1G125GW
- added U$2, U$3: MOLEX_0781710005, molex-pico-ezmate:MOLEX_0781710005
- added U$4, U$5: MOLEX_0781710003, molex-pico-ezmate:MOLEX_0781710003
- added U$6: VR42_MLB_FOOTPRINT, __temp_to_delete:VR42_MLB_FOOTPRINT
- added U$7: UBD_FOOTPRINT, __temp_to_delete:UBD_FOOTPRINT
- C16, C17: value 2.2pF -> 0.1uF
- C20: value 100nF -> 22uF; device SparkFun-Capacitors:0.1UF-0603-25V-5% -> SparkFun-Capacitors:0.22UF-0603-25V-10%
- C22: value 22uF -> 100nF; device SparkFun-Capacitors:0.22UF-0603-25V-10% -> SparkFun-Capacitors:0.1UF-0603-25V-5%
- C25, C26: value 0.1uF -> 2.2pF
- U$1: value ARGB -> VR42_MLB_FOOTPRINT; device __temp_to_delete:ARGB -> __temp_to_delete:VR42_MLB_FOOTPRINT
- renumbered U10 to M5, U5 to M0, U6 to M1, U7 to M2, U8 to M3, U9 to M4, Z1 to I32, Z10 to I41, Z11 to I42, Z12 to I43, Z13 to I21, Z14 to I22, Z15 to I23, Z16 to I24, Z17 to I25, Z18 to I26, Z19 to I27, Z2 to I33, Z20 to I28, Z21 to I29, Z22 to I30, Z23 to I31, Z24 to I10, Z25 to I11, Z26 to I12, Z27 to I13, Z28 to I14, Z29 to I15, Z3 to I34, Z30 to I16, Z31 to I17, Z32 to I18, Z33 to I19, Z34 to I20, Z35 to I2, Z36 to I3, Z37 to I4, Z38 to I5, Z39 to I6, Z4 to I35, Z40 to I7, Z41 to I8, Z42 to I9, Z5 to I36, Z6 to I37, Z7 to I38, Z8 to I39, Z9 to I40
Connections:
- removed net N$1: C1.1, U1A.VCAP_2
- removed net N$2: C2.1, U1A.VCAP_1
- removed net N$39: I21.4_DIN, I43.2_DOUT
- removed net N$61: I2.4_DIN, I20.2_DOUT
- removed net SK6803: I32.4_DIN, R12.1
- removed net SK6803_PWR: C46.1, C47.1, C48.1, C49.1, C50.1, I10.1_VDD, I11.1_VDD, I12.1_VDD, I13.1_VDD, I14.1_VDD, I15.1_VDD, I16.1_VDD, I17.1_VDD, I18.1_VDD, I19.1_VDD, I2.1_VDD, I20.1_VDD, I21.1_VDD, I22.1_VDD, I23.1_VDD, I24.1_VDD, I25.1_VDD, I26.1_VDD, I27.1_VDD, I28.1_VDD, I29.1_VDD, I3.1_VDD, I30.1_VDD, I31.1_VDD, I32.1_VDD, I33.1_VDD, I34.1_VDD, I35.1_VDD, I36.1_VDD, I37.1_VDD, I38.1_VDD, I39.1_VDD, I4.1_VDD, I40.1_VDD, I41.1_VDD, I42.1_VDD, I43.1_VDD, I5.1_VDD, I6.1_VDD, I7.1_VDD, I8.1_VDD, I9.1_VDD, U$1.V, U$14.5_VCC, U4.OUT
- new net ARGB_5V_D: I1.4_DIN, R12.1
- new net ARGB_PWR: C44.1, C46.1, C47.1, C48.1, C49.1, C50.1, I1.1_VDD, I10.1_VDD, I11.1_VDD, I12.1_VDD, I13.1_VDD, I14.1_VDD, I15.1_VDD, I16.1_VDD, I17.1_VDD, I18.1_VDD, I19.1_VDD, I2.1_VDD, I20.1_VDD, I21.1_VDD, I22.1_VDD, I23.1_VDD, I24.1_VDD, I25.1_VDD, I26.1_VDD, I27.1_VDD, I28.1_VDD, I29.1_VDD, I3.1_VDD, I30.1_VDD, I31.1_VDD, I32.1_VDD, I33.1_VDD, I34.1_VDD, I35.1_VDD, I36.1_VDD, I37.1_VDD, I38.1_VDD, I39.1_VDD, I4.1_VDD, I40.1_VDD, I41.1_VDD, I42.1_VDD, I43.1_VDD, I44.V, I5.1_VDD, I6.1_VDD, I7.1_VDD, I8.1_VDD, I9.1_VDD, LS.5_VCC, U$4.2, U$5.2, U4.OUT
- new net N$36: I31.2_DOUT, I32.4_DIN
- new net N$37: I43.2_DOUT, I44.D
- new net N$46: I1.2_DOUT, I2.4_DIN
- new net VCAP_1: C1.1, U1A.VCAP_1
- new net VCAP_2: C2.1, U1A.VCAP_2
- net ARGB_D: now also U$4.3, U$5.3
- net GND: now also C16.2, C17.2, C25.1, C26.1, I1.3_GND, I44.G, LS.!OE, LS.3_GND, U$2.1, U$3.1, U$4.1, U$5.1; no longer C16.1, C17.1, C25.2, C26.2, U$1.G, U$14.!OE, U$14.3_GND
- net LED1ST: now also LS.A_DIN; no longer U$14.A_DIN
- net MATRIX_CS: now also U$2.5, U$3.5
- net N$22: now also I20.2_DOUT, I21.4_DIN; no longer I10.4_DIN, I31.2_DOUT
- net N$3: now also I10.4_DIN; no longer U$1.D
- net N$66: now also LS.Y_DOUT; no longer C44.1, U$14.Y_DOUT
- net OSC32_I: now also C25.2; no longer C16.2
- net OSC32_O: now also C26.2; no longer C17.2
- net SPI_MISO: now also U$2.4, U$3.4
- net SPI_MOSI: now also U$2.3, U$3.3
- net VCC_1: now also C16.1, C17.1, C20.1; no longer C23.1, C25.1, C26.1
- net VCC_2: now also C23.1, U$2.2, U$3.2; no longer C20.1
