File: EAGLE/vr42/vr42-revB-kbd.sch (EAGLE design)
At the start: 176 parts, among them M0 74HC589A_DT, M1 74HC589A_DT, M2 74HC589A_DT, M3 74HC589A_DT, M4 74HC589A_DT, M5 74HC589A_DT, U1 2N7002

Commit message: Rev 1.0B
Parts:
- removed C12, C17, C18, C23: 1uF, rcl:C-EUC0603
- added CA1, CA11, CA21, CA23, CA33: 1uF, rcl:C-EUC0603
- added LOGO1: OSHW-LOGOL, random_logos:OSHW-LOGOL
- added U$3: TECSMITH-LOGOLONG, random_logos:TECSMITH-LOGOLONG
- added U$4: QMK_LOGO, random_logos:QMK_LOGO
- renumbered C10 to CA7, C11 to CA9, C13 to CA13, C14 to CA15, C15 to CA17, C16 to CA19, C19 to CA25, C20 to CA27, C21 to CA29, C22 to CA31, C24 to CA35, C25 to CA37, C26 to CA39, C27 to CA41, C28 to CA43, C7 to CA3, C8 to CA5, C9 to CA6, I1 to A1, I10 to A10, I11 to A11, I12 to A12, I13 to A13, I14 to A14, I15 to A15, I16 to A16, I17 to A17, I18 to A18, I19 to A19, I2 to A2, I20 to A20, I21 to A21, I22 to A22, I23 to A23, I24 to A24, I25 to A25, I26 to A26, I27 to A27, I28 to A28, I29 to A29, I3 to A3, I30 to A30, I31 to A31, I32 to A32, I33 to A33, I34 to A34, I35 to A35, I36 to A36, I37 to A37, I38 to A38, I39 to A39, I4 to A4, I40 to A40, I41 to A41, I42 to A42, I43 to A43, I5 to A5, I6 to A6, I7 to A7, I8 to A8, I9 to A9
Connections:
- net GND: now also CA1.2, CA11.2, CA21.2, CA23.2, CA33.2; no longer C12.2, C17.2, C18.2, C23.2
- net VCC_1: now also CA1.1, CA11.1, CA21.1, CA23.1, CA33.1; no longer C12.1, C17.1, C18.1, C23.1

Commit message: .
Parts:
- added U$5, U$6, U$7: FIDUCIAL, __temp_to_delete:FIDUCIAL
Changed lines of the file:
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@@
 <part name="U$4" library="random_logos" deviceset="QMK_LOGO" device=""/>
 <part name="LOGO1" library="random_logos" deviceset="OSHW-LOGO" device="L"/>
+<part name="U$5" library="__temp_to_delete" deviceset="FIDUCIAL" device=""/>
+<part name="U$6" library="__temp_to_delete" deviceset="FIDUCIAL" device=""/>
+<part name="U$7" library="__temp_to_delete" deviceset="FIDUCIAL" device=""/>
 </parts>
 <sheets>
@@
 <instance part="U$4" gate="G$1" x="165.1" y="15.24" smashed="yes"/>
 <instance part="LOGO1" gate="G$1" x="165.1" y="17.78" smashed="yes"/>
+<instance part="U$5" gate="G$1" x="165.1" y="7.62" smashed="yes"/>
+<instance part="U$6" gate="G$1" x="170.18" y="7.62" smashed="yes"/>
+<instance part="U$7" gate="G$1" x="175.26" y="7.62" smashed="yes"/>
 </instances>
 <busses>

Commit message: Beta 1
Parts:
- added A1.5: SK6812-E-REVERSE_V2, tecsmith_keyboards:SK6812-E-REVERSE_V2
- A1, A10, A11, A12, A13, A14, A15, A16, A17, A18, A19, A2, A20, A21, A22, A23, A24, A25, A26, A27, A28, A29, A3, A30, A31, A32, A33, A34, A35, A36, A37, A38, A39, A4, A40, A41, A42, A43, A5, A6, A7, A8, A9: value SK6812-E-REVERSE -> SK6812-E-REVERSE_V2; device ts_keyboards:SK6812-E-REVERSE -> tecsmith_keyboards:SK6812-E-REVERSE_V2
- renumbered KB_MTX to KB_MATRIX
Connections:
- removed net N$46: A1.2_DOUT, A2.4_DIN
- new net N$10: A1.2_DOUT, A1.5.4_DIN
- new net N$9: A1.5.2_DOUT, A2.4_DIN
- net GND: now also A1.5.3_GND
- net VCC_1: now also A1.5.1_VDD
Other:
- moved on the sheet: A1, ARGB
