File: EAGLE/vr42/vr42-revB-mlb.brd (EAGLE design)
At the start: 70 x 30 mm, 80 parts, among them U1 2N7002, U2 2N7002, U3 74AHCT1G125GW, U33 USB3300-EZK, U4X M25C, X1 12MHz, X2 32.768MHz, X3 24MHz

Commit message: .
Parts:
- removed J2: (no value), SparkFun-Connectors:1X02
- removed U4X: M25C, ts_kb_mcu:8-SOIC
- added EEP: M25C, ts_kb_mcu:8-SOIC
- added RST: (no value), SparkFun-Connectors:1X02
- added SWD: (no value), SparkFun-Connectors:PAD_05_03X2_TP_NO4
- added TC: (no value), __untitled:TC2030-MCP-NL
- moved LOGO1 9.91 mm to (14.8, 13.2)
- moved R8 2.00 mm to (13.0, 5.00)
- moved RGB_PD 2.00 mm to (16.0, 5.00)
- moved R7 1.98 mm to (10.9, 5.00)
- moved ARGB 1.00 mm to (45.0, 3.00)
- moved C1 1.00 mm to (65.0, 9.00)
- moved C10 1.00 mm to (15.0, 27.0)
- moved C11 1.00 mm to (21.0, 27.0)
- moved C12 1.00 mm to (23.4, 27.0)
- moved C13 1.00 mm to (29.4, 27.0)
- moved C14 1.00 mm to (20.0, 12.0)
- moved C15 1.00 mm to (33.5, 5.50)
- moved C16 1.00 mm to (32.0, 25.0)
- moved C17 1.00 mm to (40.0, 16.0)
- moved C18 1.00 mm to (67.0, 9.00)
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Connections:
- net N$2 renamed VCAP2
- net N$3 renamed VCAP1
- removed net RESET: C33.1, R18.2, STM32F405.7
- new net !RESET: C33.1, R18.2, STM32F405.7, SWD.6, TC.3
- new net SWCLK: STM32F405.49, SWD.3, TC.4
- new net SWDIO: STM32F405.46, SWD.2, TC.2
- net CS_EE: now also EEP.1; no longer U4X.1
- net GND: now also EEP.4, SWD.5, TC.5; no longer U4X.4
- net MISO: now also EEP.2; no longer U4X.2
- net MOSI: now also EEP.5; no longer U4X.5
- net N$20: now also RST.2; no longer J2.2
- net P$1: now also U$2.P$1, U$2.P$4, U$2.P$5, U$2.P$6, U$3.P$1, U$3.P$4, U$3.P$5, U$3.P$6, U$4.P$1, U$4.P$4, U$4.P$5, U$4.P$6, U$5.P$1, U$5.P$4, U$5.P$5, U$5.P$6; no longer U$2.P$10, U$2.P$7, U$2.P$8, U$2.P$9, U$3.P$10, U$3.P$7, U$3.P$8, U$3.P$9, U$4.P$10, U$4.P$7, U$4.P$8, U$4.P$9, U$5.P$10, U$5.P$7, U$5.P$8, U$5.P$9
- net SCK: now also EEP.6; no longer U4X.6
- net VCC_2: now also EEP.3, EEP.7, EEP.8, RST.1, SWD.1, TC.1; no longer J2.1, U4X.3, U4X.7, U4X.8
Routing:
- net SWCLK: track 0.00 -> 82.0 mm, vias 0 -> 3
- net SWDIO: track 0.00 -> 49.8 mm, vias 0 -> 3
- net !RESET: track 0.00 -> 43.2 mm, vias 0 -> 4
- net RESET: track 20.3 -> 0.00 mm, vias 2 -> 0
- net VCC_2: track 229.2 -> 248.9 mm, vias 18 -> 19
- net CS_MTX: track 19.7 -> 12.5 mm
- net GND: track 9.95 -> 16.4 mm, vias 47 -> 48
- net USB_SELECT: track 57.3 -> 60.0 mm
- net ARGB_DATA: track 23.7 -> 26.3 mm
- net VCC_1: track 101.2 -> 98.9 mm
- net PWR5: track 32.9 -> 31.9 mm
- net N$4: track 3.77 -> 4.49 mm
Other:
- board text added: "(c) 2024 Vino Rodrigues"
- board text added: "GND"
- board text added: "RST"
- board text added: "SWCLK"
- board text added: "SWDIO"
- board text added: "VCC"

Commit message: Rev 1.0B
Parts:
- moved LOGO1 42.1 mm to (54.8, 26.2)
Changed lines of the file:
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@@
 <setting verticaltext="up"/>
 </settings>
-<grid distance="1" unitdist="mm" unit="mm" style="lines" multiple="1" display="yes" altdistance="0.05" altunitdist="mm" altunit="mm"/>
+<grid distance="1" unitdist="mm" unit="mm" style="dots" multiple="1" display="yes" altdistance="0.1" altunitdist="mm" altunit="mm"/>
 <layers>
 <layer number="1" name="Top" color="4" fill="1" visible="yes" active="yes"/>
@@
 <wire x1="70" y1="27" x2="67" y2="30" width="0" layer="20" curve="90"/>
 <text x="62.43" y="2" size="1.5" layer="22" rot="MR0">VR42 Keyboard MLB</text>
-<text x="18" y="16" size="0.75" layer="22" rot="MR0">(c) 2024 Vino Rodrigues
+<text x="69" y="20.5" size="1.27" layer="22" rot="MR0">(c) 2024 Vino Rodrigues
 https://c1k.it/vr42</text>
 <text x="3.95" y="8" size="0.8128" layer="25" align="bottom-center">VCC</text>
@@
 <text x="5.05" y="9.55" size="0.8128" layer="26" rot="MR0" align="bottom-center">SWCLK</text>
 <text x="6.9" y="12" size="0.8128" layer="26" rot="MR0" align="bottom-center">SWDIO</text>
+<wire x1="38" y1="16" x2="42" y2="16" width="0.254" layer="22"/>
+<wire x1="42" y1="16" x2="37" y2="21" width="0.254" layer="22"/>
+<wire x1="37" y1="21" x2="42" y2="26" width="0.254" layer="22"/>
+<wire x1="42" y1="26" x2="38" y2="26" width="0.254" layer="22"/>
+<wire x1="38" y1="26" x2="35" y2="23" width="0.254" layer="22"/>
+<wire x1="35" y1="23" x2="32" y2="26" width="0.254" layer="22"/>
+<wire x1="32" y1="26" x2="28" y2="26" width="0.254" layer="22"/>
+<wire x1="28" y1="26" x2="33" y2="21" width="0.254" layer="22"/>
+<wire x1="33" y1="21" x2="28" y2="16" width="0.254" layer="22"/>
+<wire x1="28" y1="16" x2="32" y2="16" width="0.254" layer="22"/>
+<wire x1="32" y1="16" x2="35" y2="19" width="0.254" layer="22"/>
+<wire x1="35" y1="19" x2="38" y2="16" width="0.254" layer="22"/>
+<wire x1="26" y1="26" x2="26" y2="16" width="0.254" layer="22"/>
+<wire x1="26" y1="16" x2="19" y2="16" width="0.254" layer="22"/>
+<wire x1="19" y1="16" x2="19" y2="19" width="0.254" layer="22"/>
+<wire x1="19" y1="19" x2="23" y2="19" width="0.254" layer="22"/>
+<wire x1="23" y1="19" x2="23" y2="26" width="0.254" layer="22"/>
+<wire x1="23" y1="26" x2="26" y2="26" width="0.254" layer="22"/>
+<wire x1="17" y1="16" x2="17" y2="26" width="0.254" layer="22"/>
+<wire x1="17" y1="26" x2="14" y2="26" width="0.254" layer="22"/>
+<wire x1="14" y1="26" x2="14" y2="16" width="0.254" layer="22"/>
+<wire x1="14" y1="16" x2="17" y2="16" width="0.254" layer="22"/>
+<wire x1="12" y1="16" x2="9" y2="16" width="0.254" layer="22"/>
+<wire x1="9" y1="16" x2="9" y2="26" width="0.254" layer="22"/>
+<wire x1="9" y1="26" x2="12" y2="26" width="0.254" layer="22"/>
+<wire x1="12" y1="26" x2="12" y2="16" width="0.254" layer="22"/>
 </plain>
 <attributes>
@@
 <element name="U$5" library="ts_keyboards" package="MOUNTING-HOLE" value="MOUNTING-HOLE" x="67" y="3" smashed="yes"/>
 <element name="U$6" library="random_logos" package="TECSMITH-NAME" value="TECSMITH-LOGOLONG" x="62.83" y="7.7" smashed="yes" rot="MR0"/>
-<element name="LOGO1" library="random_logos" package="OSHW-LOGO-M" value="OSHW-LOGOM" x="14.75" y="13.25" smashed="yes" rot="MR0"/>
+<element name="LOGO1" library="random_logos" package="OSHW-LOGO-M" value="OSHW-LOGOM" x="54.75" y="26.25" smashed="yes" rot="MR0"/>
 <element name="TC" library="__untitled" package="TC2030-MCP-NL" value="" x="7.5" y="7" smashed="yes" rot="R270">
 <attribute name="NAME" x="7.45" y="2.5" size="1.016" layer="25" rot="R180" align="bottom-center"/>

Commit message: .
Parts:
- X1, X3: device microbuilder:CRYSTAL_2.5X2 -> __temp_to_delete:CRYSTAL_2.5X2
- X2: device adafruit2:XTAL3215 -> __temp_to_delete:CRYSTAL_2.5X2
- moved C25 0.50 mm to (52.0, 24.5)
- moved X2 0.05 mm to (26.5, 27.0)
Connections:
- net GND: now also X1.2, X1.4, X2.2, X2.4, X3.2, X3.4
- net OSC32_IN: now also X2.3; no longer X2.P$1
- net OSC32_OUT: now also X2.1; no longer X2.P$2
Routing:
- net OSC32_IN: track 8.47 -> 10.5 mm
- net N$10: track 13.5 -> 14.0 mm

Commit message: .
Parts:
- added U$7, U$8, U$9: FIDUCIAL, __temp_to_delete:FIDUCIAL
Routing:
- net GND: vias 48 -> 49
Changed lines of the file:
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@@
 <drawing>
 <settings>
-<setting alwaysvectorfont="no"/>
+<setting alwaysvectorfont="yes"/>
 <setting verticaltext="up"/>
 </settings>
-<grid distance="1" unitdist="mm" unit="mm" style="dots" multiple="1" display="yes" altdistance="0.05" altunitdist="mm" altunit="mm"/>
+<grid distance="1" unitdist="mm" unit="mm" style="dots" multiple="1" display="yes" altdistance="0.1" altunitdist="mm" altunit="mm"/>
 <layers>
 <layer number="1" name="Top" color="4" fill="1" visible="yes" active="yes"/>
@@
 <attribute name="VALUE" x="16.595" y="25.091" size="0.4064" layer="27" ratio="10"/>
 </element>
+<element name="U$7" library="__temp_to_delete" package="FIDUCIAL" value="FIDUCIAL" x="7" y="28" smashed="yes"/>
+<element name="U$9" library="__temp_to_delete" package="FIDUCIAL" value="FIDUCIAL" x="63" y="2" smashed="yes"/>
+<element name="U$8" library="__temp_to_delete" package="FIDUCIAL" value="FIDUCIAL" x="60" y="27" smashed="yes"/>
 </elements>
 <signals>
@@
 <via x="22.05" y="13.1" extent="1-16" drill="0.35"/>
 <via x="43.55" y="13" extent="1-16" drill="0.35"/>
-<via x="7" y="28" extent="1-16" drill="0.35"/>
+<via x="6.2" y="25.3" extent="1-16" drill="0.35"/>
 <via x="12.1" y="14.4" extent="1-16" drill="0.35"/>
 <via x="12" y="20.25" extent="1-16" drill="0.35"/>
@@
 <via x="42" y="21" extent="1-16" drill="0.35"/>
 <via x="39.25" y="27.85" extent="1-16" drill="0.35"/>
-<via x="63.25" y="2.85" extent="1-16" drill="0.35"/>
 <via x="66" y="22" extent="1-16" drill="0.35"/>
-<via x="62" y="26" extent="1-16" drill="0.35"/>
+<via x="61" y="25" extent="1-16" drill="0.35"/>
 <via x="58.5" y="20.55" extent="1-16" drill="0.35"/>
 <via x="55" y="10.55" extent="1-16" drill="0.35"/>
@@
 <contactref element="X2" pad="2"/>
 <contactref element="X2" pad="4"/>
+<via x="9" y="28.5" extent="1-16" drill="0.35"/>
+<via x="63.55" y="4.55" extent="1-16" drill="0.35"/>
 </signal>
 <signal name="VCC_2">

Commit message: .
Parts:
- added C34: 4,7uF, rcl:C0603
Connections:
- net GND: now also C34.2
- net VCC_2: now also C34.1
Routing:
- net VCC_2: track 249.1 -> 265.4 mm, vias 19 -> 23
- net VCC_1: track 98.9 -> 101.5 mm
- net !RESET: track 43.2 -> 41.2 mm
- net STAT_LED: track 9.75 -> 10.7 mm
- net N$18: track 7.11 -> 7.85 mm
- net SWDIO: track 49.8 -> 50.5 mm
- net N$15: track 9.19 -> 9.79 mm
Other:
- board text added: "https://c1k.it/vr42"
- board text removed: "(c) 2024 Vino Rodrigues https://c1k.it/vr42"

Commit message: Beta 1
Parts:
- renumbered EEP to EEPROM, KB_MTX to KB_MATRIX
Routing:
- net VCC_2: track 265.4 -> 264.4 mm

Commit message: .
Parts:
- removed S2: Reset, SparkFun-Switches:TACTILE_SWITCH_SMD_5.2MM
- added SW2: KMR2, 2024-11-04_19-55-01_Library:SW4_KMR221GLFS_CNK
- added TP1: TEST-POINT.3RN, tecsmith_keyboards:PAD.03X.03-RN
- D1, D2: device jlcpcb_basic_parts:SOD-123 -> tecsmith_jlcpcb_basic_parts:SOD-123
- moved RST 2.96 mm to (1.98, 17.9)
Connections:
- net GND: now also SW2.5
- net N$20: now also SW2.1, SW2.4; no longer S2.3, S2.4
- net USB_SELECT: now also TP1.1
- net VCC_2: now also SW2.2, SW2.3; no longer S2.1, S2.2
Routing:
- net N$20: track 13.2 -> 17.4 mm
- net GND: track 16.4 -> 19.1 mm, vias 49 -> 70
- net VCC_2: track 264.4 -> 266.5 mm, vias 23 -> 25
- net VCC_1: track 101.5 -> 99.6 mm, vias 5 -> 6
- net !RESET: track 41.5 -> 43.2 mm, vias 4 -> 5
- net ARGB_DATA: track 26.3 -> 27.5 mm
- net USB_SELECT: track 60.3 -> 61.1 mm
- net USB1_N: track 24.3 -> 23.5 mm
- net USB1_P: track 24.2 -> 23.4 mm
- net SWDIO: track 50.5 -> 50.1 mm, vias 3 -> 4
- net N$10: track 14.0 -> 14.1 mm, vias 0 -> 1
- added copper zone on layer 15, net GND
- added copper zone on layer 2, net GND
