File: EAGLE/vr42/vr42-revB-mlb.sch (EAGLE design)
At the start: 80 parts, among them U1 2N7002, U2 2N7002, U3 74AHCT1G125GW, U33 USB3300-EZK, U4X M25C, X1 12MHz, X2 32.768MHz, X3 24MHz

Commit message: .
Parts:
- added SWD: (no value), SparkFun-Connectors:SWD-5PIN
- added TC: (no value), __untitled:TC2030-MCP-NL
- renumbered J2 to RST, U4X to EEP
Connections:
- net N$2 renamed VCAP2
- net N$3 renamed VCAP1
- removed net RESET: C33.1, R18.2, STM32F405B.NRST
- new net !RESET: C33.1, R18.2, STM32F405B.NRST, SWD.6, TC.!RESET
- new net SWCLK: STM32F405B.PA14, SWD.3, TC.SWCLK/TCK
- new net SWDIO: STM32F405B.PA13, SWD.2, TC.SWDIO/TMS
- net GND: now also SWD.5, TC.GND
- net VCC_2: now also SWD.1, TC.VCC
Other:
- moved on the sheet: R1, R2

Commit message: .
Parts:
- X1, X3: device microbuilder:CRYSTAL2.5X2.0 -> __temp_to_delete:CRYSTAL2.5X2.0
- X2: device adafruit2:XTAL-3.2X1.5 -> __temp_to_delete:CRYSTAL2.5X2.0
Connections:
- net GND: now also X1.2, X1.4, X2.2, X2.4, X3.2, X3.4
- net N$10: now also X3.3; no longer X3.2
- net OSC32_IN: now also X2.3; no longer X2.P$1
- net OSC32_OUT: now also X2.1; no longer X2.P$2
- net OSC_IN: now also X1.3; no longer X1.2
Other:
- moved on the sheet: C11, C12, C13, R6

Commit message: .
Parts:
- added U$7, U$8, U$9: FIDUCIAL, __temp_to_delete:FIDUCIAL
Changed lines of the file:
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@@
 <part name="X3" library="__temp_to_delete" deviceset="CRYSTAL" device="2.5X2.0" value="24MHz"/>
 <part name="X1" library="__temp_to_delete" deviceset="CRYSTAL" device="2.5X2.0" value="12MHz"/>
+<part name="U$7" library="__temp_to_delete" deviceset="FIDUCIAL" device=""/>
+<part name="U$9" library="__temp_to_delete" deviceset="FIDUCIAL" device=""/>
+<part name="U$8" library="__temp_to_delete" deviceset="FIDUCIAL" device=""/>
 </parts>
 <sheets>
@@
 <attribute name="VALUE" x="92.964" y="102.87" size="1.778" layer="96"/>
 </instance>
+<instance part="U$7" gate="G$1" x="177.8" y="20.32" smashed="yes"/>
+<instance part="U$9" gate="G$1" x="187.96" y="20.32" smashed="yes"/>
+<instance part="U$8" gate="G$1" x="182.88" y="20.32" smashed="yes"/>
 </instances>
 <busses>

Commit message: .
Parts:
- added C34: 4,7uF, rcl:C-EUC0603
Connections:
- net GND: now also C34.2
- net VCC_2: now also C34.1
Changed lines of the file:
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@@
 <part name="U$9" library="__temp_to_delete" deviceset="FIDUCIAL" device=""/>
 <part name="U$8" library="__temp_to_delete" deviceset="FIDUCIAL" device=""/>
+<part name="C34" library="rcl" library_urn="urn:adsk.eagle:library:334" deviceset="C-EU" device="C0603" package3d_urn="urn:adsk.eagle:package:23616/2" value="4,7uF"/>
 </parts>
 <sheets>
@@
 <instance part="U$9" gate="G$1" x="187.96" y="20.32" smashed="yes"/>
 <instance part="U$8" gate="G$1" x="182.88" y="20.32" smashed="yes"/>
+<instance part="C34" gate="G$1" x="10.16" y="22.86" smashed="yes">
+<attribute name="NAME" x="11.684" y="23.241" size="1.778" layer="95"/>
+<attribute name="VALUE" x="11.684" y="18.161" size="1.778" layer="96"/>
+</instance>
 </instances>
 <busses>
@@
 <wire x1="30.48" y1="17.78" x2="30.48" y2="15.24" width="0.1524" layer="91"/>
 <junction x="30.48" y="15.24"/>
+<wire x1="20.32" y1="15.24" x2="10.16" y2="15.24" width="0.1524" layer="91"/>
+<junction x="20.32" y="15.24"/>
+<pinref part="C34" gate="G$1" pin="2"/>
+<wire x1="10.16" y1="15.24" x2="10.16" y2="17.78" width="0.1524" layer="91"/>
 </segment>
 <segment>
@@
 <wire x1="40.64" y1="25.4" x2="40.64" y2="27.94" width="0.1524" layer="91"/>
 <junction x="40.64" y="27.94"/>
-</segment>
-<segment>
+<wire x1="20.32" y1="27.94" x2="10.16" y2="27.94" width="0.1524" layer="91"/>
+<junction x="20.32" y="27.94"/>
+<pinref part="C34" gate="G$1" pin="1"/>
+<wire x1="10.16" y1="27.94" x2="10.16" y2="25.4" width="0.1524" layer="91"/>
+</segment>
+<segment>

Commit message: Beta 1
Parts:
- renumbered EEP to EEPROM, KB_MTX to KB_MATRIX
Changed lines of the file:
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@@
 <part name="SUPPLY20" library="SparkFun-PowerSymbols" library_urn="urn:adsk.eagle:library:530" deviceset="VCC_2" device="" value="3V3"/>
 <part name="SUPPLY23" library="supply2" library_urn="urn:adsk.eagle:library:372" deviceset="GND" device=""/>
-<part name="EEP" library="ts_kb_mcu" deviceset="M25C" device=""/>
+<part name="EEPROM" library="ts_kb_mcu" deviceset="M25C" device=""/>
 <part name="C29" library="rcl" library_urn="urn:adsk.eagle:library:334" deviceset="C-EU" device="C0603" package3d_urn="urn:adsk.eagle:package:23616/2" value="100nF"/>
 <part name="SUPPLY24" library="SparkFun-PowerSymbols" library_urn="urn:adsk.eagle:library:530" deviceset="VCC_2" device="" value="3V3"/>
@@
 <part name="SUPPLY29" library="supply2" library_urn="urn:adsk.eagle:library:372" deviceset="GND" device=""/>
 <part name="SUPPLY32" library="SparkFun-PowerSymbols" library_urn="urn:adsk.eagle:library:530" deviceset="VCC_2" device="" value="3V3"/>
-<part name="KB_MTX" library="molex-pico-ezmate" deviceset="MOLEX_0781710006" device=""/>
+<part name="KB_MATRIX" library="molex-pico-ezmate" deviceset="MOLEX_0781710006" device=""/>
 <part name="FRAME2" library="frames" library_urn="urn:adsk.eagle:library:229" deviceset="A4L-LOC" device=""/>
 <part name="ARGB" library="molex-pico-ezmate" deviceset="MOLEX_0781710003" device=""/>
@@
 <attribute name="VALUE" x="231.267" y="76.835" size="1.778" layer="96" rot="R180" align="bottom-center"/>
 </instance>
-<instance part="EEP" gate="G$1" x="132.08" y="160.02" smashed="yes">
+<instance part="EEPROM" gate="G$1" x="132.08" y="160.02" smashed="yes">
 <attribute name="NAME" x="124.46" y="165.354" size="1.778" layer="95" font="vector"/>
 <attribute name="VALUE" x="124.46" y="152.146" size="1.778" layer="96" font="vector" align="top-left"/>
@@
 <attribute name="VALUE" x="132.08" y="33.528" size="1.778" layer="96" align="bottom-center"/>
 </instance>
-<instance part="KB_MTX" gate="G$1" x="137.16" y="15.24" smashed="yes" rot="R90">
+<instance part="KB_MATRIX" gate="G$1" x="137.16" y="15.24" smashed="yes" rot="R90">
 <attribute name="VALUE" x="126.238" y="8.89" size="1.778" layer="96" font="vector" align="top-left"/>
 <attribute name="NAME" x="129.286" y="10.16" size="1.778" layer="95" font="vector" rot="R90"/>
@@
 </segment>
 <segment>
-<pinref part="EEP" gate="G$1" pin="GND"/>
+<pinref part="EEPROM" gate="G$1" pin="GND"/>
 <wire x1="121.92" y1="154.94" x2="119.38" y2="154.94" width="0.1524" layer="91"/>
 <pinref part="SUPPLY27" gate="GND" pin="GND"/>
@@
 <wire x1="124.46" y1="25.4" x2="124.46" y2="20.32" width="0.1524" layer="91"/>
 <wire x1="132.08" y1="25.4" x2="132.08" y2="22.86" width="0.1524" layer="91"/>
-<pinref part="KB_MTX" gate="G$1" pin="1"/>
+<pinref part="KB_MATRIX" gate="G$1" pin="1"/>
 </segment>
 <segment>
@@
 <wire x1="147.32" y1="22.86" x2="152.4" y2="22.86" width="0.1524" layer="91"/>
 <wire x1="147.32" y1="20.32" x2="147.32" y2="22.86" width="0.1524" layer="91"/>
-<pinref part="KB_MTX" gate="G$1" pin="M"/>
+<pinref part="KB_MATRIX" gate="G$1" pin="M"/>
 <pinref part="SUPPLY28" gate="GND" pin="GND"/>
 </segment>
@@
 <pinref part="C29" gate="G$1" pin="1"/>
 <wire x1="154.94" y1="165.1" x2="154.94" y2="162.56" width="0.1524" layer="91"/>
-<pinref part="EEP" gate="G$1" pin="VCC"/>
+<pinref part="EEPROM" gate="G$1" pin="VCC"/>
 <wire x1="154.94" y1="162.56" x2="154.94" y2="160.02" width="0.1524" layer="91"/>
-<pinref part="EEP" gate="G$1" pin="!HLD"/>
+<pinref part="EEPROM" gate="G$1" pin="!HLD"/>
 <wire x1="142.24" y1="160.02" x2="144.78" y2="160.02" width="0.1524" layer="91"/>
 <wire x1="142.24" y1="162.56" x2="144.78" y2="162.56" width="0.1524" layer="91"/>
@@
 </segment>
 <segment>
-<pinref part="EEP" gate="G$1" pin="!WP"/>
+<pinref part="EEPROM" gate="G$1" pin="!WP"/>
 <wire x1="121.92" y1="157.48" x2="119.38" y2="157.48" width="0.1524" layer="91"/>
 <pinref part="SUPPLY25" gate="G$1" pin="VCC_2"/>
@@
 <pinref part="SUPPLY32" gate="G$1" pin="VCC_2"/>
 <wire x1="134.62" y1="22.86" x2="134.62" y2="27.94" width="0.1524" layer="91"/>
-<pinref part="KB_MTX" gate="G$1" pin="2"/>
+<pinref part="KB_MATRIX" gate="G$1" pin="2"/>
 </segment>
 <segment>
@@
 <net name="MOSI" class="0">
 <segment>
-<pinref part="EEP" gate="G$1" pin="DIO"/>
+<pinref part="EEPROM" gate="G$1" pin="DIO"/>
 <wire x1="142.24" y1="154.94" x2="144.78" y2="154.94" width="0.1524" layer="91"/>
 <label x="144.78" y="154.94" size="1.27" layer="95" xref="yes"/>
@@
 <segment>
 <wire x1="137.16" y1="22.86" x2="137.16" y2="27.94" width="0.1524" layer="91"/>
-<pinref part="KB_MTX" gate="G$1" pin="3"/>
+<pinref part="KB_MATRIX" gate="G$1" pin="3"/>
 <label x="137.16" y="27.94" size="1.27" layer="95" rot="R90" xref="yes"/>
 </segment>
@@
 <net name="SCK" class="0">
 <segment>
-<pinref part="EEP" gate="G$1" pin="CLK"/>
+<pinref part="EEPROM" gate="G$1" pin="CLK"/>
 <wire x1="142.24" y1="157.48" x2="144.78" y2="157.48" width="0.1524" layer="91"/>
 <label x="144.78" y="157.48" size="1.27" layer="95" xref="yes"/>
@@
 <segment>
 <wire x1="142.24" y1="22.86" x2="142.24" y2="27.94" width="0.1524" layer="91"/>
-<pinref part="KB_MTX" gate="G$1" pin="5"/>
+<pinref part="KB_MATRIX" gate="G$1" pin="5"/>
 <label x="142.24" y="27.94" size="1.27" layer="95" rot="R90" xref="yes"/>
 </segment>
@@
 <net name="CS_EE" class="0">
 <segment>
-<pinref part="EEP" gate="G$1" pin="!CS"/>
+<pinref part="EEPROM" gate="G$1" pin="!CS"/>
 <wire x1="121.92" y1="162.56" x2="116.84" y2="162.56" width="0.1524" layer="91"/>
 <label x="116.84" y="162.56" size="1.27" layer="95" rot="R180" xref="yes"/>
@@
 <net name="MISO" class="0">
 <segment>
-<pinref part="EEP" gate="G$1" pin="DO"/>
+<pinref part="EEPROM" gate="G$1" pin="DO"/>
 <wire x1="121.92" y1="160.02" x2="116.84" y2="160.02" width="0.1524" layer="91"/>
 <label x="116.84" y="160.02" size="1.27" layer="95" rot="R180" xref="yes"/>
@@
 <segment>
 <wire x1="139.7" y1="22.86" x2="139.7" y2="27.94" width="0.1524" layer="91"/>
-<pinref part="KB_MTX" gate="G$1" pin="4"/>
+<pinref part="KB_MATRIX" gate="G$1" pin="4"/>
 <label x="139.7" y="27.94" size="1.27" layer="95" rot="R90" xref="yes"/>
 </segment>
@@
 <segment>
 <wire x1="144.78" y1="22.86" x2="144.78" y2="27.94" width="0.1524" layer="91"/>
-<pinref part="KB_MTX" gate="G$1" pin="6"/>
+<pinref part="KB_MATRIX" gate="G$1" pin="6"/>
 <label x="144.78" y="27.94" size="1.27" layer="95" rot="R90" xref="yes"/>
 </segment>

Commit message: .
Parts:
- removed S2: Reset, SparkFun-Switches:MOMENTARY-SWITCH-SPST-SMD-5.2-TALL-REDUNDANT
- added SW2: KMR2, 2024-11-04_19-55-01_Library:KMR221GLFSSW4_KMR221GLFS_CNK
- added TP1: TEST-POINT.3RN, tecsmith_keyboards:TEST-POINT.3RN
- D1, D2: device jlcpcb_basic_parts:1N5819WS -> tecsmith_jlcpcb_basic_parts:1N5819WS
Connections:
- net GND: now also SW2.5
- net N$20: now also SW2.1, SW2.4; no longer S2.2
- net USB_SELECT: now also TP1.1
- net VCC_2: now also SW2.2, SW2.3; no longer S2.1
Changed lines of the file:
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@@
 <part name="SUPPLY8" library="SparkFun-PowerSymbols" library_urn="urn:adsk.eagle:library:530" deviceset="VCC_1" device="" value="5V"/>
 <part name="LM1117" library="SparkFun-IC-Power" library_urn="urn:adsk.eagle:library:526" deviceset="V_REG_LM1117" device="SOT223" package3d_urn="urn:adsk.eagle:package:39069/1" value="AMS1117-3.3"/>
-<part name="D1" library="jlcpcb_basic_parts" deviceset="1N5819WS" device="" value="B5819W SL"/>
+<part name="D1" library="tecsmith_jlcpcb_basic_parts" deviceset="1N5819WS" device="" value="B5819W SL"/>
 <part name="SUPPLY22" library="SparkFun-PowerSymbols" library_urn="urn:adsk.eagle:library:530" deviceset="VCC_2" device="" value="3V3"/>
 <part name="SUPPLY1" library="SparkFun-PowerSymbols" library_urn="urn:adsk.eagle:library:530" deviceset="VCC_2" device="" value="3V3"/>
@@
 <part name="SUPPLY40" library="supply2" library_urn="urn:adsk.eagle:library:372" deviceset="GND" device=""/>
 <part name="SUPPLY28" library="supply2" library_urn="urn:adsk.eagle:library:372" deviceset="GND" device=""/>
-<part name="S2" library="SparkFun-Switches" deviceset="MOMENTARY-SWITCH-SPST" device="-SMD-5.2-TALL-REDUNDANT" value="Reset"/>
 <part name="RST" library="SparkFun-Connectors" library_urn="urn:adsk.eagle:library:513" deviceset="CONN_02" device="" package3d_urn="urn:adsk.eagle:package:38039/1"/>
-<part name="D2" library="jlcpcb_basic_parts" deviceset="1N5819WS" device="" value="1N4148"/>
+<part name="D2" library="tecsmith_jlcpcb_basic_parts" deviceset="1N5819WS" device="" value="1N4148"/>
 <part name="C32" library="rcl" library_urn="urn:adsk.eagle:library:334" deviceset="C-EU" device="C0603" package3d_urn="urn:adsk.eagle:package:23616/2" value="10uF"/>
 <part name="C33" library="rcl" library_urn="urn:adsk.eagle:library:334" deviceset="C-EU" device="C0603" package3d_urn="urn:adsk.eagle:package:23616/2" value="100nF"/>
@@
 <part name="U$8" library="__temp_to_delete" deviceset="FIDUCIAL" device=""/>
 <part name="C34" library="rcl" library_urn="urn:adsk.eagle:library:334" deviceset="C-EU" device="C0603" package3d_urn="urn:adsk.eagle:package:23616/2" value="4,7uF"/>
+<part name="SW2" library="2024-11-04_19-55-01_Library" deviceset="KMR221GLFS" device="SW4_KMR221GLFS_CNK" value="KMR2"/>
+<part name="SUPPLY49" library="supply2" library_urn="urn:adsk.eagle:library:372" deviceset="GND" device=""/>
+<part name="TP1" library="tecsmith_keyboards" deviceset="TEST-POINT" device=".3RN"/>
 </parts>
 <sheets>
@@
 <attribute name="NAME" x="11.684" y="23.241" size="1.778" layer="95"/>
 <attribute name="VALUE" x="11.684" y="18.161" size="1.778" layer="96"/>
+</instance>
+<instance part="TP1" gate="G$1" x="185.42" y="129.54" smashed="yes">
+<attribute name="NAME" x="182.88" y="132.08" size="1.27" layer="104"/>
 </instance>
 </instances>
@@
 <segment>
 <pinref part="USBSEL" gate="A" pin="S"/>
-<label x="182.88" y="129.54" size="1.27" layer="95" xref="yes"/>
-<wire x1="170.18" y1="129.54" x2="182.88" y2="129.54" width="0.1524" layer="91"/>
+<label x="187.96" y="129.54" size="1.27" layer="95" xref="yes"/>
+<wire x1="170.18" y1="129.54" x2="185.42" y2="129.54" width="0.1524" layer="91"/>
+<pinref part="TP1" gate="G$1" pin="1"/>
+<wire x1="185.42" y1="129.54" x2="187.96" y2="129.54" width="0.1524" layer="91"/>
+<junction x="185.42" y="129.54"/>
 </segment>
 <segment>
@@
 <attribute name="VALUE" x="233.807" y="112.395" size="1.778" layer="96" rot="R180" align="bottom-center"/>
 </instance>
-<instance part="S2" gate="G$1" x="20.32" y="137.16" smashed="yes">
-<attribute name="NAME" x="20.32" y="138.684" size="1.778" layer="95" font="vector" align="bottom-center"/>
-<attribute name="VALUE" x="20.32" y="136.652" size="1.778" layer="96" font="vector" align="top-center"/>
-</instance>
 <instance part="RST" gate="G$1" x="20.32" y="152.4" smashed="yes" rot="R270">
 <attribute name="VALUE" x="15.494" y="154.94" size="1.778" layer="96" font="vector" rot="R270"/>
@@
 <instance part="D2" gate="G$1" x="35.56" y="152.4" smashed="yes">
 <attribute name="NAME" x="33.274" y="154.305" size="1.778" layer="95"/>
-<attribute name="VALUE" x="33.274" y="148.971" size="1.778" layer="96"/>
+<attribute name="VALUE" x="34.163" y="150.114" size="1.778" layer="96" rot="R270"/>
 </instance>
 <instance part="C32" gate="G$1" x="53.34" y="147.32" smashed="yes">
@@
 <attribute name="NAME" x="134.112" y="133.604" size="1.778" layer="95" font="vector" rot="R90"/>
 <attribute name="VALUE" x="145.542" y="133.858" size="1.778" layer="96" font="vector" rot="R90" align="top-left"/>
+</instance>
+<instance part="SW2" gate="G$1" x="20.32" y="134.62" smashed="yes" rot="MR0">
+<attribute name="NAME" x="17.78" y="129.54" size="1.778" layer="95" rot="MR0"/>
+<attribute name="VALUE" x="17.78" y="127" size="1.778" layer="96" rot="MR0"/>
+</instance>
+<instance part="SUPPLY49" gate="GND" x="20.32" y="124.46" smashed="yes">
+<attribute name="VALUE" x="20.447" y="122.555" size="1.778" layer="96" rot="R180" align="bottom-center"/>
 </instance>
 </instances>
@@
 <wire x1="142.24" y1="121.92" x2="119.38" y2="121.92" width="0.1524" layer="91"/>
 </segment>
+<segment>
+<pinref part="SUPPLY49" gate="GND" pin="GND"/>
+<pinref part="SW2" gate="G$1" pin="5"/>
+<wire x1="20.32" y1="127" x2="20.32" y2="130.81" width="0.1524" layer="91"/>
+</segment>
 </net>
 <net name="PWR5" class="0">
@@
 <pinref part="SUPPLY42" gate="G$1" pin="VCC_2"/>
 <wire x1="12.7" y1="154.94" x2="12.7" y2="142.24" width="0.1524" layer="91"/>
-<pinref part="S2" gate="G$1" pin="1"/>
-<wire x1="12.7" y1="142.24" x2="12.7" y2="137.16" width="0.1524" layer="91"/>
-<wire x1="12.7" y1="137.16" x2="15.24" y2="137.16" width="0.1524" layer="91"/>
+<wire x1="12.7" y1="142.24" x2="12.7" y2="134.62" width="0.1524" layer="91"/>
 <pinref part="RST" gate="G$1" pin="1"/>
 <wire x1="20.32" y1="144.78" x2="20.32" y2="142.24" width="0.1524" layer="91"/>
 <wire x1="20.32" y1="142.24" x2="12.7" y2="142.24" width="0.1524" layer="91"/>
 <junction x="12.7" y="142.24"/>
+<pinref part="SW2" gate="G$1" pin="2"/>
+<wire x1="15.24" y1="134.62" x2="12.7" y2="134.62" width="0.1524" layer="91"/>
+<pinref part="SW2" gate="G$1" pin="3"/>
+<wire x1="15.24" y1="132.08" x2="12.7" y2="132.08" width="0.1524" layer="91"/>
+<wire x1="12.7" y1="132.08" x2="12.7" y2="134.62" width="0.1524" layer="91"/>
+<junction x="12.7" y="134.62"/>
 </segment>
 <segment>
@@
 <wire x1="22.86" y1="144.78" x2="22.86" y2="142.24" width="0.1524" layer="91"/>
 <wire x1="22.86" y1="142.24" x2="27.94" y2="142.24" width="0.1524" layer="91"/>
-<wire x1="27.94" y1="142.24" x2="27.94" y2="139.7" width="0.1524" layer="91"/>
-<pinref part="S2" gate="G$1" pin="2"/>
-<wire x1="27.94" y1="139.7" x2="27.94" y2="137.16" width="0.1524" layer="91"/>
-<wire x1="27.94" y1="137.16" x2="25.4" y2="137.16" width="0.1524" layer="91"/>
-<wire x1="27.94" y1="139.7" x2="30.48" y2="139.7" width="0.1524" layer="91"/>
-<junction x="27.94" y="139.7"/>
-<wire x1="30.48" y1="139.7" x2="30.48" y2="152.4" width="0.1524" layer="91"/>
+<wire x1="30.48" y1="142.24" x2="30.48" y2="152.4" width="0.1524" layer="91"/>
 <wire x1="30.48" y1="152.4" x2="33.02" y2="152.4" width="0.1524" layer="91"/>
 <pinref part="D2" gate="G$1" pin="A"/>
-<wire x1="30.48" y1="104.14" x2="30.48" y2="139.7" width="0.1524" layer="91"/>
-<junction x="30.48" y="139.7"/>
-</segment>
-</net>
+<wire x1="30.48" y1="104.14" x2="30.48" y2="142.24" width="0.1524" layer="91"/>
+<pinref part="SW2" gate="G$1" pin="4"/>
+<wire x1="25.4" y1="132.08" x2="27.94" y2="132.08" width="0.1524" layer="91"/>
+<wire x1="27.94" y1="132.08" x2="27.94" y2="134.62" width="0.1524" layer="91"/>
+<pinref part="SW2" gate="G$1" pin="1"/>
+<wire x1="27.94" y1="134.62" x2="27.94" y2="142.24" width="0.1524" layer="91"/>
+<wire x1="25.4" y1="134.62" x2="27.94" y2="134.62" width="0.1524" layer="91"/>
+<junction x="27.94" y="134.62"/>
+<wire x1="27.94" y1="142.24" x2="30.48" y2="142.24" width="0.1524" layer="91"/>
+<junction x="27.94" y="142.24"/>
+<junction x="30.48" y="142.24"/>
+</segment>
+</net>
